Commit message: Switched to Collada instead of STL
This allow for correct export of colors

File: urdf/nao_robot_v4.xacro (robot description, xacro)
@@ -48,5 +48,5 @@
 			<origin xyz="${xyz}" rpy="0 0 0"/>
 			<geometry name="${name}_visual_geom">
-				<mesh filename="package://nao_description/mesh/stl/${nameMesh}.stl" scale="0.1 0.1 0.1"/>
+				<mesh filename="package://nao_description/meshes/${nameMesh}.dae" scale="0.1 0.1 0.1"/>
 			</geometry>
 		</visual>
